File: Hardware/Rev 2/Sheets/Display.kicad_sch (KiCad schematic)
At the start: 7 parts

Commit message: started on pcb design
Parts:
- R? (x3): footprint Cuprum:R_0603_1608Metric -> KiCAD Library:R_0603_1608Metric
Changed lines of the file:
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@@
       (effects (font (size 1.27 1.27)) (justify right))
     )
-    (property "Footprint" "Cuprum:R_0603_1608Metric" (at 96.52 55.88 0)
+    (property "Footprint" "KiCAD Library:R_0603_1608Metric" (at 96.52 55.88 0)
       (effects (font (size 1.27 1.27)) hide)
     )
@@
       (effects (font (size 1.27 1.27)))
     )
-    (property "Footprint" "Cuprum:R_0603_1608Metric" (at 88.9 64.77 0)
+    (property "Footprint" "KiCAD Library:R_0603_1608Metric" (at 88.9 64.77 0)
       (effects (font (size 1.27 1.27)) hide)
     )
@@
       (effects (font (size 1.27 1.27)))
     )
-    (property "Footprint" "Cuprum:R_0603_1608Metric" (at 129.54 57.15 0)
-      (effects (font (size 1.27 1.27)) hide)
-    )
+    (property "Footprint" "KiCAD Library:R_0603_1608Metric" (at 129.54 57.15 0)
+      (effects (font (size 1.27 1.27)) hide)
+    )
