File: Hardware/Rev 2/Sheets/RP2040.kicad_sch (KiCad schematic)
At the start: 35 parts, among them U6 W25Q16JV, Y1 12MHz

Commit message: minor tweaks
Parts:
- added C?: 2u2, KiCAD Library:C_0603_1608Metric, symbol Device:C_Small
- R?: value 10k -> DNF
Connections:
- net +3V3: now also C?.1
- net GND: now also C?.2
Other:
- moved on the sheet: C?
Changed lines of the file:
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@@
   (junction (at 274.32 124.46) (diameter 0) (color 0 0 0 0)
   )
+  (junction (at 115.57 110.49) (diameter 0) (color 0 0 0 0)
+  )
   (junction (at 100.33 74.93) (diameter 0) (color 0 0 0 0)
   )
@@
   )
   (junction (at 80.01 30.48) (diameter 0) (color 0 0 0 0)
+  )
+  (junction (at 115.57 120.65) (diameter 0) (color 0 0 0 0)
   )
   (junction (at 97.79 40.64) (diameter 0) (color 0 0 0 0)
@@
   (no_connect (at 181.61 137.16))
   (no_connect (at 232.41 132.08))
+  (wire (pts (xy 115.57 110.49) (xy 125.73 110.49))
+    (stroke (width 0) (type default))
+  )
   (wire (pts (xy 201.93 53.34) (xy 201.93 48.26))
     (stroke (width 0) (type default))
@@
     (stroke (width 0) (type default))
   )
-  (wire (pts (xy 115.57 114.3) (xy 115.57 110.49))
+  (wire (pts (xy 115.57 113.03) (xy 115.57 110.49))
     (stroke (width 0) (type default))
   )
@@
     (stroke (width 0) (type default))
   )
+  (wire (pts (xy 125.73 118.11) (xy 125.73 120.65))
+    (stroke (width 0) (type default))
+  )
   (wire (pts (xy 163.83 83.82) (xy 181.61 83.82))
     (stroke (width 0) (type default))
@@
     (stroke (width 0) (type default))
   )
+  (wire (pts (xy 125.73 113.03) (xy 125.73 110.49))
+    (stroke (width 0) (type default))
+  )
   (wire (pts (xy 163.83 71.12) (xy 181.61 71.12))
     (stroke (width 0) (type default))
@@
     (stroke (width 0) (type default))
   )
+  (wire (pts (xy 125.73 120.65) (xy 115.57 120.65))
+    (stroke (width 0) (type default))
+  )
   (wire (pts (xy 232.41 114.3) (xy 250.19 114.3))
     (stroke (width 0) (type default))
@@
     (stroke (width 0) (type default))
   )
+  (wire (pts (xy 115.57 120.65) (xy 115.57 118.11))
+    (stroke (width 0) (type default))
+  )
   (wire (pts (xy 163.83 68.58) (xy 181.61 68.58))
     (stroke (width 0) (type default))
@@
     (stroke (width 0) (type default))
   )
-  (wire (pts (xy 115.57 120.65) (xy 115.57 119.38))
+  (wire (pts (xy 115.57 120.65) (xy 115.57 123.19))
     (stroke (width 0) (type default))
   )
@@
     )
   )
-  (symbol (lib_id "power:GND") (at 115.57 120.65 0) (unit 1)
-    (in_bom yes) (on_board yes) (dnp no) (fields_autoplaced)
-    (property "Reference" "#PWR?" (at 115.57 127 0)
-      (effects (font (size 1.27 1.27)) hide)
-    )
-    (property "Value" "GND" (at 115.57 125.2125 0)
-      (effects (font (size 1.27 1.27)))
-    )
-    (property "Footprint" "" (at 115.57 120.65 0)
-      (effects (font (size 1.27 1.27)) hide)
-    )
-    (property "Datasheet" "" (at 115.57 120.65 0)
+  (symbol (lib_id "power:GND") (at 115.57 123.19 0) (unit 1)
+    (in_bom yes) (on_board yes) (dnp no) (fields_autoplaced)
+    (property "Reference" "#PWR?" (at 115.57 129.54 0)
+      (effects (font (size 1.27 1.27)) hide)
+    )
+    (property "Value" "GND" (at 115.57 127.7525 0)
+      (effects (font (size 1.27 1.27)))
+    )
+    (property "Footprint" "" (at 115.57 123.19 0)
+      (effects (font (size 1.27 1.27)) hide)
+    )
+    (property "Datasheet" "" (at 115.57 123.19 0)
       (effects (font (size 1.27 1.27)) hide)
     )
@@
     )
   )
-  (symbol (lib_id "Device:C_Small") (at 115.57 116.84 0) (unit 1)
-    (in_bom yes) (on_board yes) (dnp no) (fields_autoplaced)
-    (property "Reference" "C?" (at 118.11 116.2113 0)
-      (effects (font (size 1.27 1.27)) (justify left))
-    )
-    (property "Value" "100n" (at 118.11 118.7513 0)
-      (effects (font (size 1.27 1.27)) (justify left))
-    )
-    (property "Footprint" "KiCAD Library:C_0603_1608Metric" (at 115.57 116.84 0)
-      (effects (font (size 1.27 1.27)) hide)
-    )
-    (property "Datasheet" "~" (at 115.57 116.84 0)
+  (symbol (lib_id "Device:C_Small") (at 115.57 115.57 0) (unit 1)
+    (in_bom yes) (on_board yes) (dnp no) (fields_autoplaced)
+    (property "Reference" "C?" (at 118.11 114.9413 0)
+      (effects (font (size 1.27 1.27)) (justify left))
+    )
+    (property "Value" "100n" (at 118.11 117.4813 0)
+      (effects (font (size 1.27 1.27)) (justify left))
+    )
+    (property "Footprint" "KiCAD Library:C_0603_1608Metric" (at 115.57 115.57 0)
+      (effects (font (size 1.27 1.27)) hide)
+    )
+    (property "Datasheet" "~" (at 115.57 115.57 0)
       (effects (font (size 1.27 1.27)) hide)
     )
@@
       (effects (font (size 1.27 1.27)) (justify right))
     )
-    (property "Value" "10k" (at 52.07 120.015 0)
+    (property "Value" "DNF" (at 52.07 120.015 0)
       (effects (font (size 1.27 1.27)) (justify right))
     )
@@
         )
       )
+    )
+  )
+  (symbol (lib_id "Device:C_Small") (at 125.73 115.57 0) (unit 1)
+    (in_bom yes) (on_board yes) (dnp no) (fields_autoplaced)
+    (property "Reference" "C?" (at 128.27 114.9413 0)
+      (effects (font (size 1.27 1.27)) (justify left))
+    )
+    (property "Value" "2u2" (at 128.27 117.4813 0)
+      (effects (font (size 1.27 1.27)) (justify left))
+    )
+    (property "Footprint" "KiCAD Library:C_0603_1608Metric" (at 125.73 115.57 0)
+      (effects (font (size 1.27 1.27)) hide)
+    )
+    (property "Datasheet" "~" (at 125.73 115.57 0)
+      (effects (font (size 1.27 1.27)) hide)
+    )
+    (pin "1")
+    (pin "2")
+    (instances
+      (project "USB-PD"
+        (path "/dbd87a35-3166-440e-a8f0-c71d214a12a6"
+          (reference "C?") (unit 1)
+        )
+        (path "/dbd87a35-3166-440e-a8f0-c71d214a12a6/e00e204b-d6fc-451e-8397-028d03c22f27"
+          (reference "C20") (unit 1)
+        )
+      )

Commit message: started on pcb design
Parts:
- R? (x10): footprint Cuprum:R_0603_1608Metric -> KiCAD Library:R_0603_1608Metric
Changed lines of the file:
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@@
       (effects (font (size 1.27 1.27)) (justify right))
     )
-    (property "Footprint" "Cuprum:R_0603_1608Metric" (at 52.07 177.8 0)
+    (property "Footprint" "KiCAD Library:R_0603_1608Metric" (at 52.07 177.8 0)
       (effects (font (size 1.27 1.27)) hide)
     )
@@
       (effects (font (size 1.27 1.27)) (justify right))
     )
-    (property "Footprint" "Cuprum:R_0603_1608Metric" (at 102.87 177.8 0)
+    (property "Footprint" "KiCAD Library:R_0603_1608Metric" (at 102.87 177.8 0)
       (effects (font (size 1.27 1.27)) hide)
     )
@@
       (effects (font (size 1.27 1.27)))
     )
-    (property "Footprint" "Cuprum:R_0603_1608Metric" (at 260.35 99.06 0)
+    (property "Footprint" "KiCAD Library:R_0603_1608Metric" (at 260.35 99.06 0)
       (effects (font (size 1.27 1.27)) hide)
     )
@@
       (effects (font (size 1.27 1.27)))
     )
-    (property "Footprint" "Cuprum:R_0603_1608Metric" (at 116.84 85.09 0)
+    (property "Footprint" "KiCAD Library:R_0603_1608Metric" (at 116.84 85.09 0)
       (effects (font (size 1.27 1.27)) hide)
     )
@@
       (effects (font (size 1.27 1.27)))
     )
-    (property "Footprint" "Cuprum:R_0603_1608Metric" (at 260.35 124.46 0)
+    (property "Footprint" "KiCAD Library:R_0603_1608Metric" (at 260.35 124.46 0)
       (effects (font (size 1.27 1.27)) hide)
     )
@@
       (effects (font (size 1.27 1.27)) (justify right))
     )
-    (property "Footprint" "Cuprum:R_0603_1608Metric" (at 43.18 177.8 0)
+    (property "Footprint" "KiCAD Library:R_0603_1608Metric" (at 43.18 177.8 0)
       (effects (font (size 1.27 1.27)) hide)
     )
@@
       (effects (font (size 1.27 1.27)))
     )
-    (property "Footprint" "Cuprum:R_0603_1608Metric" (at 40.64 118.11 0)
+    (property "Footprint" "KiCAD Library:R_0603_1608Metric" (at 40.64 118.11 0)
       (effects (font (size 1.27 1.27)) hide)
     )
@@
       (effects (font (size 1.27 1.27)) (justify right))
     )
-    (property "Footprint" "Cuprum:R_0603_1608Metric" (at 49.53 118.11 0)
+    (property "Footprint" "KiCAD Library:R_0603_1608Metric" (at 49.53 118.11 0)
       (effects (font (size 1.27 1.27)) hide)
     )
@@
       (effects (font (size 1.27 1.27)) (justify right))
     )
-    (property "Footprint" "Cuprum:R_0603_1608Metric" (at 34.29 177.8 0)
+    (property "Footprint" "KiCAD Library:R_0603_1608Metric" (at 34.29 177.8 0)
       (effects (font (size 1.27 1.27)) hide)
     )
@@
       (effects (font (size 1.27 1.27)) (justify right))
     )
-    (property "Footprint" "Cuprum:R_0603_1608Metric" (at 111.76 177.8 0)
-      (effects (font (size 1.27 1.27)) hide)
-    )
+    (property "Footprint" "KiCAD Library:R_0603_1608Metric" (at 111.76 177.8 0)
+      (effects (font (size 1.27 1.27)) hide)
+    )
