File: Hardware/Rev 2/Sheets/USB.kicad_sch (KiCad schematic)
At the start: 6 parts, among them U5 USBUF02W6

Commit message: started on pcb design
Parts:
- J?: footprint KiCAD Library:GCT_USB4110-GF-A_REVB -> Connector_USB:USB_C_Receptacle_GCT_USB4105-xx-A_16P_TopMnt_Horizontal
Changed lines of the file:
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@@
       (effects (font (size 1.27 1.27)))
     )
-    (property "Footprint" "KiCAD Library:GCT_USB4110-GF-A_REVB" (at 88.9 101.6 0)
+    (property "Footprint" "Connector_USB:USB_C_Receptacle_GCT_USB4105-xx-A_16P_TopMnt_Horizontal" (at 88.9 101.6 0)
       (effects (font (size 1.27 1.27)) hide)
     )

Commit message: small changes
Parts:
- J?: footprint Connector_USB:USB_C_Receptacle_GCT_USB4105-xx-A_16P_TopMnt_Horizontal -> KiCAD Library:GCT_USB4110-GF-A_REVB
Changed lines of the file:
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@@
       (effects (font (size 1.27 1.27)))
     )
-    (property "Footprint" "Connector_USB:USB_C_Receptacle_GCT_USB4105-xx-A_16P_TopMnt_Horizontal" (at 88.9 101.6 0)
+    (property "Footprint" "KiCAD Library:GCT_USB4110-GF-A_REVB" (at 88.9 101.6 0)
       (effects (font (size 1.27 1.27)) hide)
     )
