File: Hardware/Rev 2/Sheets/MOSFETs.kicad_sch (KiCad schematic)
At the start: 17 parts, among them Q1 PMOS, Q3 BC317, U4 INA219AxDCN

Commit message: started on pcb design
Parts:
- Q1: footprint (none) -> Package_TO_SOT_SMD:SOT-23
- Q3: footprint Package_TO_SOT_THT_AKL:TO-92_Inline_Wide_EBC -> Package_TO_SOT_SMD:SOT-23
- R? (x2): footprint Cuprum:R_0603_1608Metric -> KiCAD Library:R_0603_1608Metric
Changed lines of the file:
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@@
       (effects (font (size 1.27 1.27)) (justify left))
     )
-    (property "Footprint" "Cuprum:R_0603_1608Metric" (at 57.15 78.74 0)
+    (property "Footprint" "KiCAD Library:R_0603_1608Metric" (at 57.15 78.74 0)
       (effects (font (size 1.27 1.27)) hide)
     )
@@
       (effects (font (size 1.27 1.27)))
     )
-    (property "Footprint" "Cuprum:R_0603_1608Metric" (at 43.18 91.44 0)
+    (property "Footprint" "KiCAD Library:R_0603_1608Metric" (at 43.18 91.44 0)
       (effects (font (size 1.27 1.27)) hide)
     )
@@
       (effects (font (size 1.27 1.27)) (justify left))
     )
-    (property "Footprint" "Package_TO_SOT_THT_AKL:TO-92_Inline_Wide_EBC" (at 59.69 88.9 0)
+    (property "Footprint" "Package_TO_SOT_SMD:SOT-23" (at 59.69 88.9 0)
       (effects (font (size 1.27 1.27)) hide)
     )
@@
       (effects (font (size 1.27 1.27)))
     )
-    (property "Footprint" "" (at 74.93 68.58 0)
-      (effects (font (size 1.27 1.27)) hide)
-    )
+    (property "Footprint" "Package_TO_SOT_SMD:SOT-23" (at 74.93 68.58 0)
+      (effects (font (size 1.27 1.27)) hide)
+    )

Commit message: smaller tweaks
Parts:
- removed JP1: Bypass, Jumper:SolderJumper-2_P1.3mm_Open_RoundedPad1.0x1.5mm, symbol Jumper:SolderJumper_2_Open
Connections:
- net POW_OUT: now reaches C?.1, C?.1, C?.1, C?.1, C?.1, C?.1, J?.1 (Pin_1), J?.1 (Pin_1), J?.3 (Pin_3), J?.3 (Pin_3), J?.5 (Pin_5), J?.5 (Pin_5), R?.2, U4.2 (IN-)
Changed lines of the file:
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@@
   (junction (at 189.23 107.95) (diameter 0) (color 0 0 0 0)
   )
-  (junction (at 110.49 71.12) (diameter 0) (color 0 0 0 0)
-  )
   (junction (at 95.25 71.12) (diameter 0) (color 0 0 0 0)
   )
@@
   (junction (at 243.84 111.76) (diameter 0) (color 0 0 0 0)
   )
-  (junction (at 90.17 71.12) (diameter 0) (color 0 0 0 0)
-  )
   (junction (at 57.15 83.82) (diameter 0) (color 0 0 0 0)
   )
@@
     (stroke (width 0) (type default))
   )
-  (wire (pts (xy 90.17 60.96) (xy 90.17 71.12))
-    (stroke (width 0) (type default))
-  )
   (wire (pts (xy 57.15 83.82) (xy 57.15 86.36))
     (stroke (width 0) (type default))
@@
     (stroke (width 0) (type default))
   )
-  (wire (pts (xy 110.49 60.96) (xy 110.49 71.12))
-    (stroke (width 0) (type default))
-  )
   (wire (pts (xy 134.62 82.55) (xy 116.84 82.55))
     (stroke (width 0) (type default))
@@
     (stroke (width 0) (type default))
   )
-  (wire (pts (xy 104.14 60.96) (xy 110.49 60.96))
-    (stroke (width 0) (type default))
-  )
   (wire (pts (xy 261.62 114.3) (xy 261.62 111.76))
     (stroke (width 0) (type default))
@@
     (stroke (width 0) (type default))
   )
-  (wire (pts (xy 90.17 71.12) (xy 95.25 71.12))
-    (stroke (width 0) (type default))
-  )
   (wire (pts (xy 243.84 71.12) (xy 243.84 107.95))
     (stroke (width 0) (type default))
@@
     (stroke (width 0) (type default))
   )
-  (wire (pts (xy 105.41 71.12) (xy 110.49 71.12))
-    (stroke (width 0) (type default))
-  )
   (wire (pts (xy 168.91 119.38) (xy 179.07 119.38))
     (stroke (width 0) (type default))
@@
     (stroke (width 0) (type default))
   )
-  (wire (pts (xy 90.17 60.96) (xy 96.52 60.96))
-    (stroke (width 0) (type default))
-  )
   (wire (pts (xy 243.84 111.76) (xy 246.38 111.76))
     (stroke (width 0) (type default))
@@
     (stroke (width 0) (type default))
   )
-  (wire (pts (xy 110.49 71.12) (xy 189.23 71.12))
+  (wire (pts (xy 105.41 71.12) (xy 189.23 71.12))
     (stroke (width 0) (type default))
   )
@@
     (stroke (width 0) (type default))
   )
-  (wire (pts (xy 82.55 71.12) (xy 90.17 71.12))
+  (wire (pts (xy 82.55 71.12) (xy 95.25 71.12))
     (stroke (width 0) (type default))
   )
@@
   )
   (text "Power stage" (at 27.94 50.8 0)
+    (effects (font (size 1.27 1.27)) (justify left bottom))
+  )
+  (label "POW_OUT" (at 207.01 71.12 0) (fields_autoplaced)
     (effects (font (size 1.27 1.27)) (justify left bottom))
   )
@@
         )
       )
-    )
-  )
-  (symbol (lib_id "Jumper:SolderJumper_2_Open") (at 100.33 60.96 0) (unit 1)
-    (in_bom yes) (on_board yes) (dnp no) (fields_autoplaced)
-    (property "Reference" "JP1" (at 100.33 55.88 0)
-      (effects (font (size 1.27 1.27)))
-    )
-    (property "Value" "Bypass" (at 100.33 58.42 0)
-      (effects (font (size 1.27 1.27)))
-    )
-    (property "Footprint" "Jumper:SolderJumper-2_P1.3mm_Open_RoundedPad1.0x1.5mm" (at 100.33 60.96 0)
-      (effects (font (size 1.27 1.27)) hide)
-    )
-    (property "Datasheet" "~" (at 100.33 60.96 0)
-      (effects (font (size 1.27 1.27)) hide)
-    )
-    (pin "1")
-    (pin "2")
-    (instances
-      (project "USB-PD"
-        (path "/dbd87a35-3166-440e-a8f0-c71d214a12a6/7a5bff71-60ad-48ed-9068-6e44a60051af"
-          (reference "JP1") (unit 1)
-        )
-      )
