File: Hardware/Rev 2/USB-PD.kicad_sch (KiCad schematic)
At the start: 3 parts

Commit message: started on pcb design
Parts:
- TP1, TP2, TP3: footprint (none) -> TestPoint:TestPoint_Pad_D1.5mm
Changed lines of the file:
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@@
       (effects (font (size 1.27 1.27)) hide)
     )
-    (property "Footprint" "" (at 97.79 62.23 0)
+    (property "Footprint" "TestPoint:TestPoint_Pad_D1.5mm" (at 97.79 62.23 0)
       (effects (font (size 1.27 1.27)) hide)
     )
@@
       (effects (font (size 1.27 1.27)) hide)
     )
-    (property "Footprint" "" (at 97.79 57.15 0)
+    (property "Footprint" "TestPoint:TestPoint_Pad_D1.5mm" (at 97.79 57.15 0)
       (effects (font (size 1.27 1.27)) hide)
     )
@@
       (effects (font (size 1.27 1.27)) hide)
     )
-    (property "Footprint" "" (at 97.79 59.69 0)
+    (property "Footprint" "TestPoint:TestPoint_Pad_D1.5mm" (at 97.79 59.69 0)
       (effects (font (size 1.27 1.27)) hide)
     )

Commit message: minor work
Parts:
- removed TP1, TP2, TP3: TestPoint, TestPoint:TestPoint_Pad_D1.5mm, symbol Connector:TestPoint
Connections:
- no-connect marks 0 -> 3
Changed lines of the file:
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@@
   (junction (at 101.6 119.38) (diameter 0) (color 0 0 0 0)
   )
+  (no_connect (at 121.92 64.77))
+  (no_connect (at 121.92 62.23))
+  (no_connect (at 121.92 67.31))
   (wire (pts (xy 69.85 116.84) (xy 99.06 116.84))
     (stroke (width 0) (type default))
@@
     (stroke (width 0) (type default))
   )
-  (wire (pts (xy 97.79 62.23) (xy 121.92 62.23))
-    (stroke (width 0) (type default))
-  )
   (wire (pts (xy 238.76 139.7) (xy 256.54 139.7))
     (stroke (width 0) (type default))
@@
     (stroke (width 0) (type default))
   )
-  (wire (pts (xy 97.79 64.77) (xy 121.92 64.77))
-    (stroke (width 0) (type default))
-  )
   (wire (pts (xy 69.85 119.38) (xy 101.6 119.38))
     (stroke (width 0) (type default))
@@
     (stroke (width 0) (type default))
   )
-  (wire (pts (xy 97.79 67.31) (xy 121.92 67.31))
-    (stroke (width 0) (type default))
-  )
   (wire (pts (xy 158.75 91.44) (xy 210.82 91.44))
     (stroke (width 0) (type default))
@@
     (effects (font (size 1.27 1.27)) (justify right bottom))
   )
-  (label "RST" (at 100.33 67.31 0) (fields_autoplaced)
-    (effects (font (size 1.27 1.27)) (justify left bottom))
-  )
   (label "PD_INT_N" (at 209.55 55.88 180) (fields_autoplaced)
     (effects (font (size 1.27 1.27)) (justify right bottom))
@@
     (effects (font (size 1.27 1.27)) (justify right bottom))
   )
-  (label "SWCLK" (at 100.33 64.77 0) (fields_autoplaced)
-    (effects (font (size 1.27 1.27)) (justify left bottom))
-  )
   (label "LMOS" (at 209.55 137.16 180) (fields_autoplaced)
     (effects (font (size 1.27 1.27)) (justify right bottom))
@@
     (effects (font (size 1.27 1.27)) (justify right bottom))
   )
-  (label "SWD" (at 100.33 62.23 0) (fields_autoplaced)
-    (effects (font (size 1.27 1.27)) (justify left bottom))
-  )
   (label "USB_D-" (at 72.39 45.72 0) (fields_autoplaced)
     (effects (font (size 1.27 1.27)) (justify left bottom))
@@
   (label "SW2" (at 72.39 90.17 0) (fields_autoplaced)
     (effects (font (size 1.27 1.27)) (justify left bottom))
-  )
-  (symbol (lib_id "Connector:TestPoint") (at 97.79 67.31 90) (unit 1)
-    (in_bom yes) (on_board yes) (dnp no)
-    (property "Reference" "TP3" (at 91.44 67.31 90)
-      (effects (font (size 1.27 1.27)))
-    )
-    (property "Value" "TestPoint" (at 94.488 64.77 90)
-      (effects (font (size 1.27 1.27)) hide)
-    )
-    (property "Footprint" "TestPoint:TestPoint_Pad_D1.5mm" (at 97.79 62.23 0)
-      (effects (font (size 1.27 1.27)) hide)
-    )
-    (property "Datasheet" "~" (at 97.79 62.23 0)
-      (effects (font (size 1.27 1.27)) hide)
-    )
-    (pin "1")
-    (instances
-      (project "USB-PD"
-        (path "/dbd87a35-3166-440e-a8f0-c71d214a12a6"
-          (reference "TP3") (unit 1)
-        )
-      )
-    )
   )
   (symbol (lib_name "VBUS_1") (lib_id "power:VBUS") (at 203.2 147.32 0) (unit 1)
@@
         )
       )
-    )
-  )
-  (symbol (lib_id "Connector:TestPoint") (at 97.79 62.23 90) (unit 1)
-    (in_bom yes) (on_board yes) (dnp no)
-    (property "Reference" "TP1" (at 91.44 62.23 90)
-      (effects (font (size 1.27 1.27)))
-    )
-    (property "Value" "TestPoint" (at 94.488 59.69 90)
-      (effects (font (size 1.27 1.27)) hide)
-    )
-    (property "Footprint" "TestPoint:TestPoint_Pad_D1.5mm" (at 97.79 57.15 0)
-      (effects (font (size 1.27 1.27)) hide)
-    )
-    (property "Datasheet" "~" (at 97.79 57.15 0)
-      (effects (font (size 1.27 1.27)) hide)
-    )
-    (pin "1")
-    (instances
-      (project "USB-PD"
-        (path "/dbd87a35-3166-440e-a8f0-c71d214a12a6"
-          (reference "TP1") (unit 1)
-        )
-      )
-    )
-  )
-  (symbol (lib_id "Connector:TestPoint") (at 97.79 64.77 90) (unit 1)
-    (in_bom yes) (on_board yes) (dnp no)
-    (property "Reference" "TP2" (at 91.44 64.77 90)
-      (effects (font (size 1.27 1.27)))
-    )
-    (property "Value" "TestPoint" (at 94.488 62.23 90)
-      (effects (font (size 1.27 1.27)) hide)
-    )
-    (property "Footprint" "TestPoint:TestPoint_Pad_D1.5mm" (at 97.79 59.69 0)
-      (effects (font (size 1.27 1.27)) hide)
-    )
-    (property "Datasheet" "~" (at 97.79 59.69 0)
-      (effects (font (size 1.27 1.27)) hide)
-    )
-    (pin "1")
-    (instances
-      (project "USB-PD"
-        (path "/dbd87a35-3166-440e-a8f0-c71d214a12a6"
-          (reference "TP2") (unit 1)
-        )
-      )
