File: Hardware/Rev 2/USB-PD.kicad_pcb (KiCad board)
At the start: 2 copper layers, 54.1 x 45.1 mm, 84 parts, among them IC1 MCP1792T, J1 USB4110-GF-A_REVB, J2 R 2.54 mm, J3 L 2.54 mm, Q1 PMOS, Q2 BC817, Q3 BC317, SW1 SW_MENU, SW2 SW_DOWN, SW3 SW_CONF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

Commit message: small changes
Parts:
- J1: footprint Connector_USB:USB_C_Receptacle_GCT_USB4105-xx-A_16P_TopMnt_Horizontal -> KiCAD Library:GCT_USB4110-GF-A_REVB
- moved U6 61.0 mm to (130.1, 100.8), turned to -90 degrees
- moved SW3 43.4 mm to (127.1, 88.0)
- moved SW2 37.1 mm to (152.1, 88.0)
- moved SW1 30.4 mm to (139.6, 88.0)
- moved J1 1.66 mm to (139.6, 89.3)
- moved U2 0.16 mm to (139.5, 103.8), turned to -90 degrees
Routing:
- net /RP2040/QSPI_SS: track 0.00 -> 14.7 mm
- net /RP2040/QSPI_SD1: track 0.00 -> 13.1 mm
- net /RP2040/QSPI_SD2: track 0.00 -> 11.7 mm
- net /RP2040/QSPI_SD3: track 0.00 -> 10.1 mm
- net /RP2040/QSPI_SCLK: track 0.00 -> 8.61 mm
- net /RP2040/QSPI_SD0: track 0.00 -> 7.22 mm
- net /LCD_CS: track 6.02 -> 2.31 mm
- net /LCD_D/C: track 5.40 -> 1.87 mm
- net /LCD_SCK: track 5.59 -> 2.74 mm
- net /LCD_MOSI: track 4.85 -> 3.17 mm
- net /LCD_RST: track 5.00 -> 3.60 mm

Commit message: minor work
Parts:
- removed TP1, TP2, TP3: TestPoint, TestPoint:TestPoint_Pad_D1.5mm
- moved C38 72.1 mm to (156.4, 102.3)
- moved C39 72.1 mm to (156.4, 104.3)
- moved R15 67.5 mm to (145.2, 104.2), turned to -90 degrees
- moved Y1 61.9 mm to (147.2, 103.4), turned to -90 degrees
- moved R5 61.8 mm to (148.8, 96.4)
- moved R7 61.4 mm to (148.8, 98.9), turned to 0 degrees
- moved R4 59.6 mm to (148.8, 97.7), turned to 0 degrees
- moved R16 57.3 mm to (127.0, 100.8), turned to -90 degrees
- moved SW4 56.2 mm to (124.4, 100.8), turned to -90 degrees
- moved Q2 55.6 mm to (151.9, 97.7), turned to -90 degrees
- moved RN1 25.7 mm to (111.2, 157.1)
- moved RN2 25.7 mm to (107.0, 157.1)
- moved U1 25.7 mm to (110.8, 142.1)
- moved U5 25.7 mm to (104.1, 172.1)
- moved D1 25.7 mm to (117.4, 144.1)
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Connections:
- U2 pad 24: /SWCLK -> /RP2040/SWCLK
- U2 pad 25: /SWD -> /RP2040/SWD
- U2 pad 26: /RST -> /RP2040/RUN
Routing:
- net /LCD_BL: track 0.00 -> 30.6 mm
- net /LCD_D/C: track 1.87 -> 11.6 mm, vias 0 -> 1
- net /LCD_CS: track 2.31 -> 11.5 mm, vias 0 -> 1
- net /LCD_RST: track 3.60 -> 10.8 mm, vias 0 -> 1
- net /LCD_MOSI: track 3.17 -> 9.97 mm, vias 0 -> 1
- net /LCD_SCK: track 2.74 -> 9.51 mm, vias 0 -> 1
- net /RP2040/XIN: track 0.00 -> 6.43 mm
- net Net-(R16-Pad2): track 0.00 -> 5.05 mm
- net GND: track 0.00 -> 4.70 mm, vias 0 -> 2
- net /Display/BL_CTR: track 0.00 -> 3.83 mm, vias 0 -> 1
- net /RP2040/QSPI_SS: track 14.7 -> 17.3 mm
- net Net-(Q2-C): track 0.00 -> 2.45 mm
- net /RP2040/XOUT: track 0.00 -> 2.34 mm
- net Net-(C38-Pad2): track 0.00 -> 1.77 mm
- net Net-(Q2-B): track 0.00 -> 1.50 mm

Commit message: smaller tweaks
Parts:
- removed JP1: Bypass, Jumper:SolderJumper-2_P1.3mm_Open_RoundedPad1.0x1.5mm
- moved C18 110.5 mm to (177.6, 96.3)
- moved C19 110.5 mm to (177.6, 98.2)
- moved C21 110.5 mm to (177.6, 100.2)
- moved C1 110.2 mm to (203.2, 84.0)
- moved C17 110.2 mm to (194.3, 84.0)
- moved C11 110.2 mm to (197.7, 89.8)
- moved C13 110.2 mm to (197.7, 104.9)
- moved C23 110.2 mm to (197.7, 106.9)
- moved C24 110.2 mm to (197.7, 108.8)
- moved C26 110.2 mm to (202.7, 115.0)
- moved C27 110.2 mm to (202.7, 117.0)
- moved C28 110.2 mm to (197.7, 112.7)
- moved C29 110.2 mm to (197.7, 114.7)
- moved C30 110.2 mm to (197.7, 116.6)
- moved C37 110.2 mm to (190.8, 84.0)
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Connections:
- net Net-(J2-Pin_1) renamed /MOSFETs/POW_OUT
Routing:
- net /LCD_BL: track 30.6 -> 9.69 mm
- net Net-(Q1-G): track 0.00 -> 16.3 mm, vias 0 -> 2
- net +3V3: track 0.00 -> 15.5 mm
- net /I2C0_SCL: track 0.00 -> 14.1 mm
- net /Display/BL_CTR: track 3.83 -> 16.8 mm
- net /I2C0_SDA: track 0.00 -> 13.0 mm
- net +1V1: track 2.40 -> 12.0 mm
- net /MOSFETs/POW_OUT: track 0.00 -> 7.13 mm
- net /RP2040/XIN: track 6.43 -> 0.00 mm
- net /RP2040/QSPI_SD3: track 10.1 -> 15.7 mm
- net /RP2040/QSPI_SCLK: track 8.61 -> 14.2 mm
- net /CC2: track 0.00 -> 5.37 mm
- net Net-(D3-A): track 0.00 -> 5.37 mm
- net /CC1: track 0.00 -> 4.14 mm
- net /PD_SDA: track 0.00 -> 4.10 mm
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- added copper zone on B.Cu, net /MOSFETs/POW_OUT
- added copper zone on F.Cu, net GND
- added copper zone on B.Cu, net Net-(D3-A)
- added copper zone on B.Cu, net VBUS
